File: From Programmer's Reference Guide/C64.sch (EAGLE design)
At the start: 239 parts, among them CN2 USERPORT-C64-EDGE, CN3 CASSETTEPORT, CN4 MAB6H, CN5 MAB8SH, CN6 EXPANSIONPORT, CN7 MAB7SH, Q1 tp29b, Q2 2N4401, Q3 2N3904, Q4 2N2222, Q5 2N2222, Q6 2N2222, Q7 2N2222, Q8 2N2222, SW1 9077-2, U1 6526, U10 4164, U11 4164, U12 4164, U13 74LS257N, U14 74LS258N, U15 74LS139N, U16 4066, U17 C64PLA, U18 6581, U19 6569, U2 6526, U20 556DIGITAL, U21 4164, U22 4164, U23 4164, U24 4164, U25 74LS257N, U26 74LS373N, U27 74LS08N, U28 4066, U29 74LS74N, U3 2364, U30 74LS193N, U31 74629, U32 MC4044, U4 2364, U5 2332, U6 2114, U7 6510, U8 7406N, U9 4164, Y1 17.73 MHz

Commit message: zone 1 done
Parts:
- added C76: 0.1 uF, 326298_rev_a:CAPACITOR_12_03_07C_0309/12
- added R15: 1.5 K, 326298_rev_a:RESISTOR_12_03_07R_0307/12
- added R18: 230, 326298_rev_a:RESISTOR_12_03_07R_0307/12
- added R46: 2.1 K, 326298_rev_a:R_0307/12R_0307/12
- C1, C10, C11, C16, C18, C2, C29, C3, C30, C31, C32, C33, C35, C37, C4, C44, C45, C46, C47, C48, C49, C5, C50, C51, C52, C53, C54, C59, C6, C7, C89, C9, C92, C93, C95, C96: device rcl:C-EU075-032X103 -> 326298_rev_a:C_0307/12C_0309/12
- C100, C20, C21, C97, C98, C99: device rcl:C-EU075-032X103 -> 326298_rev_a:C_0203
- C101: device rcl:C-EU075-032X103 -> 326298_rev_a:CAPACITOR_6_03_8.5
- C12, C13, C15, C17, C34, C57, C62, C8, C94: device rcl:CPOL-EUE3.5-10 -> 326298_rev_a:C_E_2,5-6
- C14, C24, C64, C65: device rcl:CPOL-EUE3.5-10 -> 326298_rev_a:CAPACITOR_ELECTROLYTIC_2.5_6
- C19, C88, C90: device rcl:CPOL-EUE3.5-10 -> 326298_rev_a:E37-31.5-17.5-E
- C22, C23, C25, C26, C27, C28, C38, C39, C41, C42, C43: device rcl:C-EU075-032X103 -> 326298_rev_a:CAPACITOR_12_3_7C_0309/12
- C36, C55, C56, C58, C60, C68, C71, C72, C73, C74, C77, C78, C79, C80, C81, C82, C83, C84, C85, C86, C87: device rcl:C-EU075-032X103 -> 326298_rev_a:CAPACITOR_12_03_07C_0309/12
- C40: value 0.22 uF -> 10 uF 25V; device rcl:C-EU075-032X103 -> 326298_rev_a:CAPACITOR_12_3_7C_0309/12
- C61, C63, C66, C67: device rcl:C-EU075-032X103 -> 326298_rev_a:CAPACITOR_15_04_10
- C91: device rcl:CPOL-EUE3.5-10 -> 326298_rev_a:C_E_5-9
- CN1: device con-lstb:MA20-1 -> 326298_rev_a:MA20-1
- CN2: device 0RB_Commodore:USERPORT-C64-EDGE -> 326298_rev_a:USERPORT-C64-EDGE
- CN3: device 0RB_Commodore:CASSETTEPORT -> 326298_rev_a:CASSETTEPORT
- CN4: value MAB6H -> DIN6; device con-hirschmann:MAB6H -> 326298_rev_a:DIN6
- CN5: value MAB8SH -> DIN5; device con-hirschmann:MAB8SH -> 326298_rev_a:DIN5
- CN6: device 0RB_Commodore:EXPANSIONPORT-C64 -> 326298_rev_a:EXPANSIONPORT-C64
- CN8, CN9: device con-subd:M09H -> 326298_rev_a:CONTROL_PORT
- CR1, CR2: device diode:ZENER-DIODEDO34-7 -> 326298_rev_a:ZD_0307/12
- CR3: device 0RB_Passive:DIODE-S -> 326298_rev_a:D_0307/12
- CR4: value (none) -> BRIDGE_RECTIFIERS; device rectifier:S41 -> 326298_rev_a:BRIDGE_RECTIFIERS
- CR5, CR6: device diode:1N4004 -> 326298_rev_a:D_0307/12
- F1: device fuse:SH32 -> 326298_rev_a:SH32
- FB1, FB10, FB11, FB12, FB14, FB15, FB16, FB17, FB18, FB2, FB20, FB21, FB3, FB4, FB5, FB6: value FERRIT -> (none); device 0RB_Passive:FERRIT -> 326298_rev_a:FB_0307/12R_0307/12
- FB7, FB9: value FERRIT -> (none); device 0RB_Passive:FERRIT -> 326298_rev_a:FERRITE_BEAD_12_3_7R_0307/12
- FB8: value FERRIT -> (none); device 0RB_Passive:FERRIT -> 326298_rev_a:RESISTOR_12_3_7R_0307/12
- L1, L2, L3: device 0RB_Passive:COIL -> 326298_rev_a:INDUCTOR_12_3_7
- L4: value (none) -> LINEFILTER; device wuerth-elektronik:WE-CMB_M -> 326298_rev_a:LINEFILTER
- L5: device 0RB_Passive:COIL -> 326298_rev_a:COIL
- Q1: device transistor:-NPN-TO220 -> 326298_rev_a:TIP29B
- Q2: device transistor:2N4416 -> 326298_rev_a:2N4401
- Q3: device transistor:2N4416 -> 326298_rev_a:2N3904
- Q4, Q5, Q6, Q7: value 2N2222 -> PN2222; device transistor-small-signal:2N2222 -> 326298_rev_a:PN2222
- Q8: value 2N2222 -> PN2222; device transistor-npn:2N2222 -> 326298_rev_a:PN2222
- R1, R2, R3, R37, R39, R4, R41, R43, R44, R45, R5, R6, R7: device rcl:R-EU_0204/2V -> 326298_rev_a:R_0307/12R_0307/12
- R10, R11, R13, R14, R16, R17, R19, R20, R21, R22, R23, R24, R26, R8, R9: device rcl:R-EU_0204/2V -> 326298_rev_a:RESISTOR_12_03_07R_0307/12
- R25, R27: device pot:TRIM_EU-CA6H -> 326298_rev_a:POT_METER
- R28, R29, R30, R31, R33, R34, R35, R36, R38, R42: device rcl:R-EU_0204/2V -> 326298_rev_a:RESISTOR_12_3_7R_0307/12
- RF1: device 0RB_Commodore:RF-MODULATOR -> 326298_rev_a:RF-MODULATOR
- RP1, RP2: device resistor-sil:E4R -> 326298_rev_a:RESISTOR_PACK_4
- RP3: device 0RB_Passive:RP8 -> 326298_rev_a:RP8
- RP4: device 0RB_Passive:RP9 -> 326298_rev_a:RP9
- SW1: value 9077-2 -> DPDT_SWITCH; device switch-misc:9077-2 -> 326298_rev_a:DPDT_SWITCH
- U1, U2: device 0RB_65xx:6526 -> 326298_rev_a:6526
- U10, U11, U12, U21, U22, U23, U24, U9: device 0RB_Memory:4164 -> 326298_rev_a:4164
- U13, U25: device 74xx-us:74LS257N -> 326298_rev_a:74LS257N
- U14: device 74xx-us:74LS258N -> 326298_rev_a:74LS258N
- U15: device 74xx-us:74LS139N -> 326298_rev_a:74LS139N
- U16, U28: device 0RB_CMOS:4066 -> 326298_rev_a:4066
- U17: device 0RB_Commodore:C64PLA -> 326298_rev_a:C64PLA
- U18: device 0RB_65xx:6581 -> 326298_rev_a:6581
- U19: device 0RB_65xx:6569 -> 326298_rev_a:6569
- U20: device 0RB_Lineair:556DIGITAL -> 326298_rev_a:556DIGITAL
- U26: device 74xx-us:74LS373N -> 326298_rev_a:74LS373N
- U27: device 74xx-us:74LS08N -> 326298_rev_a:74LS08N
- U29: device 74xx-us:74LS74N -> 326298_rev_a:74LS74N
- U3, U4: device 0RB_Memory:2364 -> 326298_rev_a:2364
- U30: device 0RB_TTL:74LS193N -> 326298_rev_a:74LS193N
- U31: device 0RB_TTL:74629 -> 326298_rev_a:74629
- U32: device 0RB_IC:MC4044 -> 326298_rev_a:MC4044
- U6: device memory:2114 -> 326298_rev_a:2114
- U7: device 0RB_65xx:6510 -> 326298_rev_a:6510
- U8: value 7406N -> SN7406NN; device 74xx-us:7406N -> 326298_rev_a:SN7406NN
- VR1: value 7812T -> VR; device linear:7812T -> 326298_rev_a:VR
- VR2: value 7805T -> VR; device linear:7805T -> 326298_rev_a:VR
Connections:
- new net N$143: C76.1, R15.1, U31G$1.RNG
- net +12V: now also C57.1, C62.1, C94.1; no longer C57.+, C62.+, C94.+
- net +5V: now also C64.1, C65.1; no longer C64.+, C65.+
- net D0: now also U7>NAME.D0; no longer U7>NAME.DB0
- net D1: now also U7>NAME.D1; no longer U7>NAME.DB1
- net D2: now also U7>NAME.D2; no longer U7>NAME.DB2
- net D3: now also U7>NAME.D3; no longer U7>NAME.DB3
- net D4: now also U7>NAME.D4; no longer U7>NAME.DB4
- net D5: now also U7>NAME.D5; no longer U7>NAME.DB5
- net D6: now also U7>NAME.D6; no longer U7>NAME.DB6
- net D7: now also U7>NAME.D7; no longer U7>NAME.DB7
- net GND: now also C14.2, C15.2, C17.2, C19.2, C24.2, C34.2, C57.2, C62.2, C64.2, C65.2, C76.2, C8.2, C88.2, C91.2, C94.2, R15.2; no longer C14.+, C15.-, C17.-, C19.-, C24.-, C34.-, C57.-, C62.-, C64.-, C65.-, C8.-, C88.-, C91.-, C94.-, CN4.PE, CN4.PE@1, CN5.PE, CN5.PE@1, U31G$1.RNG
- net IRQ: now also U19G$2.!IRQ!, U1G$1.!IRQ!, U7>NAME.!IRQ!; no longer U19G$2.IRQ, U1G$1./IRQ, U7>NAME./IRQ
- net N$1: now also C12.1; no longer C12.+
- net N$10: now also C13.2; no longer C13.-
- net N$11: now also C12.2; no longer C12.-
- net N$120: now also U2G$1.!PC!; no longer U2G$1./PC
- net N$129: now also U2G$1.!FLAG!; no longer U2G$1./FLAG
- net N$141: now also U7>NAME.CLKOUT; no longer U7>NAME.PHI2
- net N$163: now also U19G$2.!CS!; no longer U19G$2.CS
- net N$171: now also U1G$1.!FLAG!; no longer U1G$1./FLAG
- net N$182: now also U1G$1.!CS!; no longer U1G$1./CS
- net N$183: now also U2G$1.!CS!; no longer U2G$1./CS
- net N$19: now also L4.4; no longer L4.1
- net N$21: now also L4.2; no longer L4.4
- net N$22: now also L4.1; no longer L4.2
- net N$24: now also C90.2; no longer C90.-
- net N$25: now also C19.1; no longer C19.+
- net N$26: now also C90.1; no longer C90.+
- net N$27: now also C88.1; no longer C88.+
- net N$33: now also R18.1
- net N$5: now also C13.1; no longer C13.+
- net N$53: now also U19G$2.!CAS!; no longer U19G$2.CAS
- net N$55: now also U19G$2.!RAS!; no longer U19G$2.RAS
- net N$58: now also C24.1; no longer C24.+
- net NMI: now also U2G$1.!IRQ!, U7>NAME.!NMI!; no longer U2G$1./IRQ, U7>NAME./NMI
- net PHI0: now also U7>NAME.CLKIN; no longer U7>NAME.PHI0
- net PHI2: now also U18G$2.CLKOUT, U1G$1.CLKOUT, U2G$1.CLKOUT; no longer U18G$2.PHI2, U1G$1.PHI2, U2G$1.PHI2
- net RES: now also U1G$1.!RES!, U2G$1.!RES!, U7>NAME.!RES!; no longer U1G$1./RES, U2G$1./RES, U7>NAME./RES
- net RW: now also R46.1, U19G$2.!R/W!; no longer U19G$2.R/W
- net VCC: now also C14.1, C15.1, C17.1, C34.1, C8.1, C91.1, R46.2; no longer C14.-, C15.+, C17.+, C34.+, C8.+, C91.+
Other:
- moved on the sheet: C14, C40, C90, RF1
